Commit message: Holy jesus simulation

File: betabot_ws/src/betabot_description/urdf/betabot.urdf (robot description, URDF)
Before this commit: robot betabot, 3 links, 2 joints
Links:
- added link battery, mass 25.0; collision mesh filename=battery.stl scale=0.01 0.01 0.01; visual mesh filename=battery.stl scale=0.01 0.01 0.01
- link chassis: geometry collision mesh filename=body.stl name=body scale=0.01 0.01 0.01; visual mesh filename=body.stl name=body scale=0.01 0.01 0.01
- link left_wheel: geometry collision mesh filename=left_wheel.stl name=left_wheel scale=0.01 0.01 0.01; visual mesh filename=left_wheel.stl name=left_wheel scale=0.01 0.01 0.01
- link right_wheel: geometry collision mesh filename=right_wheel.stl name=right_wheel scale=0.01 0.01 0.01; visual mesh filename=right_wheel.stl name=right_wheel scale=0.01 0.01 0.01
Joints:
- added joint battery_hinge: type continuous, parent chassis, child battery, origin xyz=0 0 0 rpy=0 0 0, axis 0 1 0, limit effort=10000 velocity=1000
- joint left_wheel_hinge: origin xyz=0 0.15 0 rpy=0 0 0 -> xyz=0 0 0.0 rpy=0 0 0
- joint right_wheel_hinge: origin xyz=0 -0.15 0 rpy=0 0 0 -> xyz=0 0 0.0 rpy=0 0 0

Commit message: So good

File: betabot_ws/src/betabot_description/urdf/betabot.urdf (robot description, URDF)
Before this commit: robot betabot, 4 links, 3 joints
Links:
- added link top, mass 5.0; collision mesh filename=top.stl scale=0.01 0.01 0.01; visual mesh filename=top.stl scale=0.01 0.01 0.01
Joints:
- added joint top_hinge: type continuous, parent chassis, child top, origin xyz=0 0 0 rpy=0 0 0, axis 0 1 0, limit effort=10000 velocity=1000

Commit message: Added simulator

File: betabot_ws/src/betabot_description/urdf/betabot.urdf (robot description, URDF)
Before this commit: robot betabot, 5 links, 4 joints
Joints:
- removed joint left_wheel_hinge
- removed joint right_wheel_hinge
- added joint left_wheel_joint: type continuous, parent chassis, child left_wheel, origin xyz=0 0 0.0 rpy=0 0 0, axis 0 1 0, limit effort=10000 velocity=1000
- added joint right_wheel_joint: type continuous, parent chassis, child right_wheel, origin xyz=0 0 0.0 rpy=0 0 0, axis 0 1 0, limit effort=10000 velocity=1000

Commit message: Dance baby dance

File: betabot_ws/src/betabot_description/urdf/betabot.urdf (robot description, URDF)
Before this commit: robot betabot, 5 links, 4 joints
Joints:
- joint left_wheel_joint: origin xyz=0 0 0.0 rpy=0 0 0 -> xyz=0 0 0.7 rpy=0 0 0
- joint right_wheel_joint: origin xyz=0 0 0.0 rpy=0 0 0 -> xyz=0 0 0.7 rpy=0 0 0

Commit message: Combine simulator and robot

File: betabot_ws/src/betabot_description/urdf/betabot.urdf (robot description, URDF)
Before this commit: robot betabot, 5 links, 4 joints
Links:
- link chassis: mass 15.0 -> 50.0
