Commit message: Update simulator

File: ros/src/betabot_description/urdf/betabot.urdf (robot description, URDF)
Before this commit: robot betabot, 5 links, 4 joints
Links:
- removed link battery
- removed link top
- link chassis: mass 50.0 -> 40
- link left_wheel: mass 5 -> 10
- link right_wheel: mass 5 -> 10
Joints:
- removed joint battery_hinge
- removed joint top_hinge
- joint left_wheel_joint: limit effort=10000 velocity=1000 -> effort=10 velocity=10; origin xyz=0 0 0.7 rpy=0 0 0 -> xyz=0 0 0 rpy=0 0 0
- joint right_wheel_joint: limit effort=10000 velocity=1000 -> effort=10 velocity=10; origin xyz=0 0 0.7 rpy=0 0 0 -> xyz=0 0 0 rpy=0 0 0

Commit message: Update with feet, fix float int

File: ros/src/betabot_description/urdf/betabot.urdf (robot description, URDF)
Before this commit: robot betabot, 3 links, 2 joints
Links:
- removed link left_wheel
- removed link right_wheel
- added link left_foot, mass 0.1; collision mesh filename=left_foot.stl name=left_foot scale=0.01 0.01 0.01; visual mesh filename=left_foot.stl name=left_foot scale=0.01 0.01 0.01
- added link right_foot, mass 0.1; collision mesh filename=right_foot.stl name=right_foot scale=0.01 0.01 0.01; visual mesh filename=right_foot.stl name=right_foot scale=0.01 0.01 0.01
- link chassis: mass 40 -> 1
Joints:
- removed joint left_wheel_joint
- removed joint right_wheel_joint
- added joint left_foot_joint: type continuous, parent chassis, child left_foot, origin xyz=0 0 0 rpy=0 0 0, axis 0 1 0, limit effort=10 velocity=10
- added joint right_foot_joint: type continuous, parent chassis, child right_foot, origin xyz=0 0 0 rpy=0 0 0, axis 0 1 0, limit effort=10 velocity=10

Commit message: Legs!

File: ros/src/betabot_description/urdf/betabot.urdf (robot description, URDF)
Before this commit: robot betabot, 3 links, 2 joints
Links:
- added link left_leg, mass 0.1; collision mesh filename=left_leg.stl name=left_leg scale=0.01 0.01 0.01; visual mesh filename=left_leg.stl name=left_leg scale=0.01 0.01 0.01
- added link right_leg, mass 0.1; collision mesh filename=right_leg.stl name=right_leg scale=0.01 0.01 0.01; visual mesh filename=right_leg.stl name=right_leg scale=0.01 0.01 0.01
Joints:
- added joint left_leg_joint: type continuous, parent chassis, child left_leg, origin xyz=0 0 0 rpy=0 0 0, axis 0 1 0, limit effort=10 velocity=10
- added joint right_leg_joint: type continuous, parent chassis, child right_leg, origin xyz=0 0 0 rpy=0 0 0, axis 0 1 0, limit effort=10 velocity=10

Commit message: Legs

File: ros/src/betabot_description/urdf/betabot.urdf (robot description, URDF)
Before this commit: robot betabot, 5 links, 4 joints
Links:
- added link left_lower_leg, mass 0.1; collision mesh filename=left_lower_leg.stl name=left_lower_leg scale=0.01 0.01 0.01; visual mesh filename=left_lower_leg.stl name=left_lower_leg scale=0.01 0.01 0.01
- added link left_motor, mass 0.8; collision mesh filename=left_motor.stl name=left_motor scale=0.01 0.01 0.01; visual mesh filename=left_motor.stl name=left_motor scale=0.01 0.01 0.01
- added link right_lower_leg, mass 0.1; collision mesh filename=right_lower_leg.stl name=right_lower_leg scale=0.01 0.01 0.01; visual mesh filename=right_lower_leg.stl name=right_lower_leg scale=0.01 0.01 0.01
- added link right_motor, mass 0.8; collision mesh filename=right_motor.stl name=right_motor scale=0.01 0.01 0.01; visual mesh filename=right_motor.stl name=right_motor scale=0.01 0.01 0.01
Joints:
- added joint left_lower_leg_joint: type continuous, parent left_leg, child left_lower_leg, origin xyz=0 0 0 rpy=0 0 0, axis 0 1 0, limit effort=10 velocity=10
- added joint left_motor_joint: type continuous, parent chassis, child left_motor, origin xyz=0 0 0 rpy=0 0 0, axis 0 1 0, limit effort=10 velocity=10
- added joint right_lower_leg_joint: type continuous, parent right_leg, child right_lower_leg, origin xyz=0 0 0 rpy=0 0 0, axis 0 1 0, limit effort=10 velocity=10
- added joint right_motor_joint: type continuous, parent chassis, child right_motor, origin xyz=0 0 0 rpy=0 0 0, axis 0 1 0, limit effort=10 velocity=10
- joint left_foot_joint: parent chassis -> left_lower_leg
- joint right_foot_joint: parent chassis -> right_lower_leg

Commit message: Dancing

File: ros/src/betabot_description/urdf/betabot.urdf (robot description, URDF)
Before this commit: robot betabot, 9 links, 8 joints
Joints:
- removed joint left_leg_joint
- removed joint left_lower_leg_joint
- removed joint right_leg_joint
- removed joint right_lower_leg_joint
- added joint left_hip_joint: type continuous, parent chassis, child left_leg, origin xyz=0 0 0 rpy=0 0 0, axis 0 1 0, limit effort=10 velocity=10
- added joint left_knee_joint: type continuous, parent left_leg, child left_lower_leg, origin xyz=0 0 0 rpy=0 0 0, axis 0 1 0, limit effort=10 velocity=10
- added joint right_hip_joint: type continuous, parent chassis, child right_leg, origin xyz=0 0 0 rpy=0 0 0, axis 0 1 0, limit effort=10 velocity=10
- added joint right_knee_joint: type continuous, parent right_leg, child right_lower_leg, origin xyz=0 0 0 rpy=0 0 0, axis 0 1 0, limit effort=10 velocity=10

Commit message: Sim legs!

File: ros/src/betabot_description/urdf/betabot.urdf (robot description, URDF)
Before this commit: robot betabot, 9 links, 8 joints
Joints:
- joint left_knee_joint: origin xyz=0 0 0 rpy=0 0 0 -> xyz=0.25 0 -0.7 rpy=0 0 0
- joint right_knee_joint: origin xyz=0 0 0 rpy=0 0 0 -> xyz=0.25 0 -0.7 rpy=0 0 0

Commit message: Fixed feet

File: ros/src/betabot_description/urdf/betabot.urdf (robot description, URDF)
Before this commit: robot betabot, 9 links, 8 joints
Joints:
- joint left_foot_joint: origin xyz=0 0 0 rpy=0 0 0 -> xyz=-0.5 0 -0.7 rpy=0 0 0
- joint right_foot_joint: origin xyz=0 0 0 rpy=0 0 0 -> xyz=-0.5 0 -0.7 rpy=0 0 0
